File: driver_list.kicad_sch (KiCad schematic)
At the start: 54 parts

Commit message: major pcb update
Parts:
- renumbered R16 to R24, R17 to R25, R18 to R26, R19 to R27, R20 to R28, R21 to R29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
