File: VacuumIndicatorDynamic.kicad_sch (KiCad schematic)
At the start: 42 parts, among them J1 Conn_01x02_Male, J2 Conn_01x03_Male, J3 Conn_01x03_Male, J4 Conn_01x03_Male, SW1 SW_DIP_x01, SW2 SW_DIP_x01, SW3 SW_DIP_x01, SW4 SW_DIP_x01, U1 AP1117-25, U2 YAAJ_BluePill

Commit message: update pcb
Connections:
- net AU3: now also U2.17 (PB9); no longer U2.11 (PB3)
- net AU4: now also U2.16 (PB8); no longer U2.12 (PB4)
- net AU5: now also U2.15 (PB7); no longer U2.13 (PB5)
- net AU7: now also U2.13 (PB5); no longer U2.15 (PB7)
- net AU8: now also U2.12 (PB4); no longer U2.16 (PB8)
- net AU9: now also U2.11 (PB3); no longer U2.17 (PB9)
Changed lines of the file:
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@@
+    (effects (font (size 1.27 1.27)) (justify right bottom))
+  )
+  (label "AU5" (at 165.1 63.5 180)
     (effects (font (size 1.27 1.27)) (justify right bottom))
   )
@@
   (label "AU2" (at 205.74 35.56 0)
     (effects (font (size 1.27 1.27)) (justify left bottom))
+  )
+  (label "AU9" (at 165.1 53.34 180)
+    (effects (font (size 1.27 1.27)) (justify right bottom))
   )
   (label "K5" (at 97.79 158.75 0)
@@
     (effects (font (size 1.27 1.27)) (justify left bottom))
   )
+  (label "AU7" (at 165.1 58.42 180)
+    (effects (font (size 1.27 1.27)) (justify right bottom))
+  )
   (label "TX1" (at 262.89 27.94 0)
     (effects (font (size 1.27 1.27)) (justify left bottom))
@@
     (effects (font (size 1.27 1.27)) (justify left bottom))
   )
-  (label "AU4" (at 165.1 55.88 180)
-    (effects (font (size 1.27 1.27)) (justify right bottom))
-  )
   (label "K6" (at 165.1 35.56 180)
-    (effects (font (size 1.27 1.27)) (justify right bottom))
-  )
-  (label "AU8" (at 165.1 66.04 180)
     (effects (font (size 1.27 1.27)) (justify right bottom))
   )
@@
     (effects (font (size 1.27 1.27)) (justify left bottom))
   )
+  (label "AU8" (at 165.1 55.88 180)
+    (effects (font (size 1.27 1.27)) (justify right bottom))
+  )
   (label "A5" (at 66.04 64.77 0)
     (effects (font (size 1.27 1.27)) (justify left bottom))
@@
     (effects (font (size 1.27 1.27)) (justify right bottom))
   )
-  (label "AU3" (at 165.1 53.34 180)
-    (effects (font (size 1.27 1.27)) (justify right bottom))
-  )
-  (label "AU5" (at 165.1 58.42 180)
-    (effects (font (size 1.27 1.27)) (justify right bottom))
-  )
   (label "A6" (at 69.85 64.77 0)
     (effects (font (size 1.27 1.27)) (justify left bottom))
-  )
-  (label "AU9" (at 165.1 68.58 180)
-    (effects (font (size 1.27 1.27)) (justify right bottom))
   )
   (label "TX1" (at 165.1 40.64 180)
@@
   )
   (label "AU3" (at 143.51 109.22 180)
-    (effects (font (size 1.27 1.27)) (justify right bottom))
-  )
-  (label "AU7" (at 165.1 63.5 180)
     (effects (font (size 1.27 1.27)) (justify right bottom))
   )
@@
     (effects (font (size 1.27 1.27)) (justify left bottom))
   )
+  (label "AU4" (at 165.1 66.04 180)
+    (effects (font (size 1.27 1.27)) (justify right bottom))
+  )
+  (label "AU3" (at 165.1 68.58 180)
+    (effects (font (size 1.27 1.27)) (justify right bottom))
+  )
   (label "AU1" (at 143.51 104.14 180)

Commit message: remove copper area add mounting holes
Other:
- note added: "External VCC 5V connector"
- note added: "connector for 5v vcc switch"
Changed lines of the file:
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@@
     (stroke (width 0) (type default) (color 0 0 0 0))
   )
+  (text "External VCC 5V connector\n" (at 50.8 52.07 0)
+    (effects (font (size 1.27 1.27)) (justify left bottom))
+  )
+  (text "connector for 5v vcc switch\n" (at 73.66 16.51 0)
+    (effects (font (size 1.27 1.27)) (justify left bottom))
+  )
   (label "K2" (at 205.74 30.48 0)
     (effects (font (size 1.27 1.27)) (justify left bottom))
@@
     (effects (font (size 1.27 1.27)) (justify right bottom))
   )
+  (label "External +24V Q=0.1-0.4 connector" (at 120.65 67.31 0)
+    (effects (font (size 1.27 1.27)) (justify left bottom))
+  )
   (label "AU5" (at 143.51 114.3 180)

Commit message: several pcb updates
Parts:
- C3: footprint Capacitor_THT:C_Axial_L5.1mm_D3.1mm_P7.50mm_Horizontal -> Capacitor_SMD:C_0805_2012Metric
- C4: footprint Capacitor_THT:CP_Axial_L10.0mm_D6.0mm_P15.00mm_Horizontal -> Capacitor_SMD:C_0805_2012Metric
- C5: footprint Capacitor_THT:CP_Axial_L10.0mm_D6.0mm_P15.00mm_Horizontal -> Capacitor_THT:CP_Radial_D8.0mm_P5.00mm
Changed lines of the file:
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@@
       (effects (font (size 1.27 1.27)) (justify left))
     )
-    (property "Footprint" "Capacitor_THT:CP_Axial_L10.0mm_D6.0mm_P15.00mm_Horizontal" (id 2) (at 123.19 45.72 0)
+    (property "Footprint" "Capacitor_THT:CP_Radial_D8.0mm_P5.00mm" (id 2) (at 123.19 45.72 0)
       (effects (font (size 1.27 1.27)) hide)
     )
@@
       (effects (font (size 1.27 1.27)) (justify left))
     )
-    (property "Footprint" "Capacitor_THT:C_Axial_L5.1mm_D3.1mm_P7.50mm_Horizontal" (id 2) (at 96.52 45.72 0)
+    (property "Footprint" "Capacitor_SMD:C_0805_2012Metric" (id 2) (at 96.52 45.72 0)
       (effects (font (size 1.27 1.27)) hide)
     )
@@
       (effects (font (size 1.27 1.27)) (justify left))
     )
-    (property "Footprint" "Capacitor_THT:CP_Axial_L10.0mm_D6.0mm_P15.00mm_Horizontal" (id 2) (at 110.49 45.72 0)
+    (property "Footprint" "Capacitor_SMD:C_0805_2012Metric" (id 2) (at 110.49 45.72 0)
       (effects (font (size 1.27 1.27)) hide)
     )
@@
     )
     (path "/84d05990-c8b5-4a92-8244-f6de53abe747"
-      (reference "C3") (unit 1) (value "1n") (footprint "Capacitor_THT:C_Axial_L5.1mm_D3.1mm_P7.50mm_Horizontal")
+      (reference "C3") (unit 1) (value "1n") (footprint "Capacitor_SMD:C_0805_2012Metric")
     )
     (path "/f1fda711-2596-45d6-ba24-29f1f5117356"
-      (reference "C4") (unit 1) (value "100n") (footprint "Capacitor_THT:CP_Axial_L10.0mm_D6.0mm_P15.00mm_Horizontal")
+      (reference "C4") (unit 1) (value "100n") (footprint "Capacitor_SMD:C_0805_2012Metric")
     )
     (path "/83217fd8-a53a-4d04-ba20-b54a75754205"
-      (reference "C5") (unit 1) (value "47uF") (footprint "Capacitor_THT:CP_Axial_L10.0mm_D6.0mm_P15.00mm_Horizontal")
+      (reference "C5") (unit 1) (value "47uF") (footprint "Capacitor_THT:CP_Radial_D8.0mm_P5.00mm")
     )
     (path "/40dfc85e-6e54-4324-b21c-0117d1a04406"

Commit message: major pcb update
Parts:
- added R10, R14, R15, R16, R20, R21, R8, R9: 47k, Resistor_SMD:R_0805_2012Metric, symbol Device:R
- renumbered R6 to R11, R7 to R12, R11 to R13, R10 to R17, R12 to R18, R13 to R19, R14 to R22, R15 to R23, R8 to R6, R9 to R7, VT5 to VT4, VT4 to VT5
Connections:
- net +24V: now also R10.1, R14.1, R15.1, R16.1, R20.1, R21.1, R8.1, R9.1
- net +2V5: now also EL1.2 (Накал_2_+); no longer EL1.1 (Накал_1)
- net AU1: now also U2.11 (PB3); no longer U2.33 (PB0)
- net AU2: now also U2.12 (PB4); no longer U2.34 (PB1)
- net AU3: now also U2.13 (PB5); no longer U2.17 (PB9)
- net AU4: now also U2.14 (PB6); no longer U2.16 (PB8)
- net AU6: now also U2.16 (PB8); no longer U2.14 (PB6)
- net AU7: now also U2.17 (PB9); no longer U2.13 (PB5)
- net AU8: now also U2.34 (PB1); no longer U2.12 (PB4)
- net AU9: now also U2.33 (PB0); no longer U2.11 (PB3)
- net S_OUT_1: now reaches EL1.12 (Cетка_1), VT2.3 (C)
- net S_OUT_1: now also R8.2
- net S_OUT_2: now reaches EL1.13 (Сетка_2), VT5.3 (C)
- net S_OUT_2: now also R14.2
- net S_OUT_3: now reaches EL1.14 (Сетка_3), VT6.3 (C)
- net S_OUT_3: now also R15.2
- net S_OUT_4: now reaches EL1.15 (Сетка_4), VT8.3 (C)
- net S_OUT_4: now also R20.2
- net S_OUT_5: now reaches EL1.16 (Сетка_5), VT9.3 (C)
- net S_OUT_5: now also R21.2
- net S_OUT_6: now reaches EL1.17 (Сетка_6), VT7.3 (C)
- net S_OUT_6: now also R16.2
- net S_OUT_7: now reaches EL1.18 (Сетка_7), VT4.3 (C)
- net S_OUT_7: now also R10.2
- net S_OUT_8: now reaches EL1.19 (Сетка_8), VT3.3 (C)
- net S_OUT_8: now also R9.2
- net at VT1.3 (C): now also EL1.1 (Накал/Катод_1_-); no longer EL1.2 (Накал_2)
- net K1 renamed S1
- net K2 renamed S2
- net K3 renamed S3
- net K4 renamed S4
- net K5 renamed S5
- net K6 renamed S6
- net K7 renamed S7
- net K8 renamed S8
Other:
- moved on the sheet: R11, R12, R13, R17, R18, R19, R22, R23, R5, VT1, VT2, VT3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

Commit message: Remake sch after fabrication. Clear repo
Parts:
- removed BT1: Battery_Cell, Connector_PinHeader_2.54mm:PinHeader_1x02_P2.54mm_Vertical, symbol Device:Battery_Cell
- removed C1: 10uF, Capacitor_THT:CP_Radial_D6.3mm_P2.50mm, symbol pspice:CAP
- removed C2: 22uF, Capacitor_THT:CP_Radial_D6.3mm_P2.50mm, symbol pspice:CAP
- removed C3: 1n, Capacitor_SMD:C_0805_2012Metric, symbol pspice:CAP
- removed C4: 100n, Capacitor_SMD:C_0805_2012Metric, symbol pspice:CAP
- removed C5: 47uF, Capacitor_THT:CP_Radial_D8.0mm_P5.00mm, symbol pspice:CAP
- removed D1: LED, LED_SMD:LED_0805_2012Metric, symbol Device:LED
- removed EL1: VacuumIndicator, ProjectLibrary:VauumIndicator_ILC_8-9, symbol ProjectLib:VacuumIndicator
- removed J1: Conn_01x02_Male, Connector_PinHeader_2.54mm:PinHeader_1x02_P2.54mm_Vertical, symbol Connector:Conn_01x02_Male
- removed J2, J3, J4: Conn_01x03_Male, Connector_PinHeader_2.54mm:PinHeader_1x03_P2.54mm_Vertical, symbol Connector:Conn_01x03_Male
- removed R1, R4, R6, R7: 10k, Resistor_SMD:R_0805_2012Metric, symbol Device:R
- removed R10, R14, R15, R16, R20, R21, R8, R9: 47k, Resistor_SMD:R_0805_2012Metric, symbol Device:R
- removed R11, R12, R13, R17, R18, R19, R22, R23, R3: 4.7k, Resistor_SMD:R_0805_2012Metric, symbol Device:R
- removed R2: R_Photo, Resistor_THT:R_Axial_DIN0204_L3.6mm_D1.6mm_P1.90mm_Vertical, symbol Device:R_Photo
- removed R5: 1k, Resistor_SMD:R_0805_2012Metric, symbol Device:R
- removed SW1: SW_DIP_x01, Connector_PinSocket_2.54mm:PinSocket_1x02_P2.54mm_Vertical, symbol Switch:SW_DIP_x01
- removed SW2, SW3, SW4: SW_DIP_x01, Button_Switch_SMD:SW_SPST_FSMSM, symbol Switch:SW_DIP_x01
- removed U1: AP1117-25, Package_TO_SOT_SMD:SOT-223-3_TabPin2, symbol Regulator_Linear:AP1117-25
- removed U2: YAAJ_BluePill, ProjectLibrary:YAAJ_BluePill_1, symbol ProjectLib:YAAJ_BluePill
- removed VT1, VT2, VT3, VT4, VT5, VT6, VT7, VT8, VT9: KT3102AM, Package_TO_SOT_THT:TO-92_HandSolder, symbol ProjectLib:KT3102AM
Connections:
- no-connect marks 12 -> 0
Other:
- removed sheet AnodeDriverList
- added sheet Connectors (Connectors.kicad_sch)
- added sheet Driver (Driver.kicad_sch)
- added sheet Indicator (Indicator.kicad_sch)
- added sheet Interface (Interface.kicad_sch)
- added sheet Logic Level Converter (LLC.kicad_sch)
- added sheet MCU (MCU.kicad_sch)
- added sheet Power Managment (Power.kicad_sch)
- added sheet Power Managment1 (Power.kicad_sch)
- note removed: "External VCC 5V connector"
- note removed: "connector for 5v vcc switch"
